Commit message: Update main.urdf

File: udm_urdf/urdf/main.urdf (robot description, URDF)
Before this commit: robot hand, 16 links, 15 joints
Links:
- removed link index_distal_phalange
- removed link index_intermediate_phalange
- removed link index_proximal_phalange
- removed link map
- removed link middle_distal_phalange
- removed link middle_intermediate_phalange
- removed link middle_proximal_phalange
- removed link pinky_distal_phalange
- removed link pinky_intermediate_phalange
- removed link pinky_proximal_phalange
- removed link ring_distal_phalange
- removed link ring_intermediate_phalange
- removed link ring_proximal_phalange
- removed link thumb_distal_phalange
- removed link thumb_proximal_phalange
- added link index_phalange_base; visual cylinder length=0.03 radius=0.01
- added link index_phalange_end; visual cylinder length=0.025 radius=0.005
- added link index_phalange_middle; visual cylinder length=0.025 radius=0.008
- added link middle_phalange_base; visual cylinder length=0.03 radius=0.01
- added link middle_phalange_end; visual cylinder length=0.03 radius=0.005
- added link middle_phalange_middle; visual cylinder length=0.03 radius=0.008
- added link pinky_phalange_base; visual cylinder length=0.02 radius=0.005
- added link pinky_phalange_end; visual cylinder length=0.02 radius=0.005
- added link pinky_phalange_middle; visual cylinder length=0.02 radius=0.005
- added link ring_phalange_base; visual cylinder length=0.03 radius=0.01
- added link ring_phalange_end; visual cylinder length=0.025 radius=0.005
- added link ring_phalange_middle; visual cylinder length=0.025 radius=0.008
- added link thumb_phalange_base; visual cylinder length=0.03 radius=0.01
- added link thumb_phalange_end; visual cylinder length=0.02 radius=0.008
- link base_link: geometry visual box size=0.08 0.03 0.10
Joints:
- removed joint hand
- removed joint hand_to_index_proximal
- removed joint hand_to_middle_proximal
- removed joint hand_to_pinky_proximal
- removed joint hand_to_ring_proximal
- removed joint hand_to_thumb_proximal
- removed joint index_intermediate_to_index_distal
- removed joint index_proximal_to_index_intermediate
- removed joint middle_intermediate_to_middle_distal
- removed joint middle_proximal_to_middle_intermediate
- removed joint pinky_intermediate_to_pinky_distal
- removed joint pinky_proximal_to_pinky_intermediate
- removed joint ring_intermediate_to_ring_distal
- removed joint ring_proximal_to_ring_intermediate
- removed joint thumb_proximal_to_thumb_distal
- added joint base_link_to_index_base: type revolute, parent base_link, child index_phalange_base, origin xyz=0.03 0.0 0.05, axis 1 0 0, limit lower=-1.65 upper=1.57 effort=1000 velocity=0.5
- added joint base_link_to_middle_base: type revolute, parent base_link, child middle_phalange_base, origin xyz=0.008 0.0 0.05, axis 1 0 0, limit lower=-1.65 upper=1.57 effort=1000 velocity=0.5
- added joint base_link_to_pinky_base: type revolute, parent base_link, child pinky_phalange_base, origin xyz=-0.035 0.0 0.05, axis 1 0 0, limit lower=-1.65 upper=1.57 effort=1000 velocity=0.5
- added joint base_link_to_ring_base: type revolute, parent base_link, child ring_phalange_base, origin xyz=-0.015 0.0 0.05, axis 1 0 0, limit lower=-1.65 upper=1.57 effort=1000 velocity=0.5
- added joint index_base_to_middle: type revolute, parent index_phalange_base, child index_phalange_middle, origin xyz=0.0 0.0 0.03, axis 1 0 0, limit lower=-1.65 upper=0 effort=1000 velocity=0.5
- added joint index_middle_to_end: type revolute, parent index_phalange_middle, child index_phalange_end, origin xyz=0.0 0.0 0.025, axis 1 0 0, limit lower=-1.57 upper=0 effort=1000 velocity=0.5
- added joint middle_base_to_middle: type revolute, parent middle_phalange_base, child middle_phalange_middle, origin xyz=0.0 0.0 0.03, axis 1 0 0, limit lower=-1.65 upper=0 effort=1000 velocity=0.5
- added joint middle_middle_to_end: type revolute, parent middle_phalange_middle, child middle_phalange_end, origin xyz=0.0 0.0 0.03, axis 1 0 0, limit lower=-1.57 upper=0 effort=1000 velocity=0.5
- added joint pinky_base_to_middle: type revolute, parent pinky_phalange_base, child pinky_phalange_middle, origin xyz=0.0 0.0 0.02, axis 1 0 0, limit lower=-1.65 upper=0 effort=1000 velocity=0.5
- added joint pinky_middle_to_end: type revolute, parent pinky_phalange_middle, child pinky_phalange_end, origin xyz=0.0 0.0 0.02, axis 1 0 0, limit lower=-1.57 upper=0 effort=1000 velocity=0.5
- added joint ring_base_to_middle: type revolute, parent ring_phalange_base, child ring_phalange_middle, origin xyz=0.0 0.0 0.03, axis 1 0 0, limit lower=-1.65 upper=0 effort=1000 velocity=0.5
- added joint ring_middle_to_end: type revolute, parent ring_phalange_middle, child ring_phalange_end, origin xyz=0.0 0.0 0.025, axis 1 0 0, limit lower=-1.57 upper=0 effort=1000 velocity=0.5
- added joint thumb_base_palm: type revolute, parent base_link, child thumb_phalange_base, origin xyz=0.04 0 -0.025 rpy=0 1.57 0, axis 1 0 0, limit lower=-1.57 upper=0 effort=1000 velocity=0.5
- added joint thumb_end_to_thumb_base: type revolute, parent thumb_phalange_base, child thumb_phalange_end, origin xyz=0 0 0.03 rpy=0 0 0, axis 1 0 0, limit lower=-1.0 upper=0 effort=1000 velocity=0.5
